Commit message: Updated URDF file

File: models/spot.urdf (robot description, URDF)
Before this commit: robot spot, 13 links, 12 joints
Links:
- link base_link: mass 11.44 -> 16.7; geometry collision mesh filename=package://spot_IL/models/meshes/base.obj; visual mesh filename=package://spot_IL/models/meshes/base.obj
- link front_left.hip: mass 2.145 -> 2.5; geometry collision mesh filename=package://spot_IL/models/meshes/fl.hip.obj; visual mesh filename=package://spot_IL/models/meshes/fl.hip.obj
- link front_left.lowerleg: mass 0.715 -> 0.8; geometry collision mesh filename=package://spot_IL/models/meshes/fr.lleg.obj; visual mesh filename=package://spot_IL/models/meshes/fr.lleg.obj
- link front_left.upperleg: mass 1.43 -> 1.8; geometry collision mesh filename=package://spot_IL/models/meshes/fl.uleg.obj; visual mesh filename=package://spot_IL/models/meshes/fl.uleg.obj
- link front_right.hip: mass 2.145 -> 2.5; geometry collision mesh filename=package://spot_IL/models/meshes/fr.hip.obj; visual mesh filename=package://spot_IL/models/meshes/fr.hip.obj
- link front_right.lowerleg: mass 0.715 -> 0.8; geometry collision mesh filename=package://spot_IL/models/meshes/fr.lleg.obj; visual mesh filename=package://spot_IL/models/meshes/fr.lleg.obj
- link front_right.upperleg: mass 1.43 -> 1.8; geometry collision mesh filename=package://spot_IL/models/meshes/fr.uleg.obj; visual mesh filename=package://spot_IL/models/meshes/fr.uleg.obj
- link hind_left.hip: mass 2.145 -> 2.5; geometry collision mesh filename=package://spot_IL/models/meshes/hl.hip.obj; visual mesh filename=package://spot_IL/models/meshes/hl.hip.obj
- link hind_left.lowerleg: mass 0.715 -> 0.8; geometry collision mesh filename=package://spot_IL/models/meshes/hl.lleg.obj; visual mesh filename=package://spot_IL/models/meshes/hl.lleg.obj
- link hind_left.upperleg: mass 1.43 -> 1.8; geometry collision mesh filename=package://spot_IL/models/meshes/hl.uleg.obj; visual mesh filename=package://spot_IL/models/meshes/hl.uleg.obj
- link hind_right.hip: mass 2.145 -> 2.5; geometry collision mesh filename=package://spot_IL/models/meshes/hr.hip.obj; visual mesh filename=package://spot_IL/models/meshes/hr.hip.obj
- link hind_right.lowerleg: mass 0.715 -> 0.8; geometry collision mesh filename=package://spot_IL/models/meshes/hr.lleg.obj; visual mesh filename=package://spot_IL/models/meshes/hr.lleg.obj
- link hind_right.upperleg: mass 1.43 -> 1.8; geometry collision mesh filename=package://spot_IL/models/meshes/hr.uleg.obj; visual mesh filename=package://spot_IL/models/meshes/hr.uleg.obj
Joints:
- joint front_left.hx: limit lower=-0.78539816339744827899 upper=0.78539816339744827899 effort=1000 velocity=1000.00 -> lower=-0.785 upper=0.785 effort=100 velocity=2.00
- joint front_left.hy: limit lower=-0.89884456477707963539 upper=2.2951079663725435509 effort=1000 velocity=1000.00 -> lower=-0.898 upper=2.295 effort=100 velocity=2.00
- joint front_left.knee: limit lower=-2.7929 upper=-0.254402 effort=1000 velocity=1000.00 -> lower=-2.792 upper=-0.254 effort=100 velocity=2.00
- joint front_right.hx: limit lower=-0.78539816339744827899 upper=0.78539816339744827899 effort=1000 velocity=1000.00 -> lower=-0.785 upper=0.785 effort=100 velocity=2.00
- joint front_right.hy: limit lower=-0.898845 upper=2.24363 effort=1000 velocity=1000.00 -> lower=-0.898 upper=2.295 effort=100 velocity=2.00
- joint front_right.knee: limit lower=-2.7929 upper=-0.255648 effort=1000 velocity=1000.00 -> lower=-2.792 upper=-0.255 effort=100 velocity=2.00
- joint hind_left.hx: limit lower=-0.78539816339744827899 upper=0.78539816339744827899 effort=1000 velocity=1000.00 -> lower=-0.785 upper=0.785 effort=100 velocity=2.00
- joint hind_left.hy: limit lower=-0.89884456477707963539 upper=2.2951079663725435509 effort=1000 velocity=1000.00 -> lower=-0.898 upper=2.295 effort=100 velocity=2.00
- joint hind_left.knee: limit lower=-2.7929 upper=-0.247067 effort=1000 velocity=1000.00 -> lower=-2.792 upper=-0.247 effort=100 velocity=2.00
- joint hind_right.hx: limit lower=-0.78539816339744827899 upper=0.78539816339744827899 effort=1000 velocity=1000.00 -> lower=-0.785 upper=0.785 effort=100 velocity=2.00
- joint hind_right.hy: limit lower=-0.89884456477707963539 upper=2.2951079663725435509 effort=1000 velocity=1000.00 -> lower=-0.898 upper=2.295 effort=100 velocity=2.00
- joint hind_right.knee: limit lower=-2.7929 upper=-0.248282 effort=1000 velocity=1000.00 -> lower=-2.792 upper=-0.248 effort=100 velocity=2.00

Commit message: Rename the package

File: models/spot.urdf (robot description, URDF)
Before this commit: robot spot, 13 links, 12 joints
Links:
- link base_link: geometry collision mesh filename=package://spot_IL_environment/models/meshes/base.obj; visual mesh filename=package://spot_IL_environment/models/meshes/base.obj
- link front_left.hip: geometry collision mesh filename=package://spot_IL_environment/models/meshes/fl.hip.obj; visual mesh filename=package://spot_IL_environment/models/meshes/fl.hip.obj
- link front_left.lowerleg: geometry collision mesh filename=package://spot_IL_environment/models/meshes/fr.lleg.obj; visual mesh filename=package://spot_IL_environment/models/meshes/fr.lleg.obj
- link front_left.upperleg: geometry collision mesh filename=package://spot_IL_environment/models/meshes/fl.uleg.obj; visual mesh filename=package://spot_IL_environment/models/meshes/fl.uleg.obj
- link front_right.hip: geometry collision mesh filename=package://spot_IL_environment/models/meshes/fr.hip.obj; visual mesh filename=package://spot_IL_environment/models/meshes/fr.hip.obj
- link front_right.lowerleg: geometry collision mesh filename=package://spot_IL_environment/models/meshes/fr.lleg.obj; visual mesh filename=package://spot_IL_environment/models/meshes/fr.lleg.obj
- link front_right.upperleg: geometry collision mesh filename=package://spot_IL_environment/models/meshes/fr.uleg.obj; visual mesh filename=package://spot_IL_environment/models/meshes/fr.uleg.obj
- link hind_left.hip: geometry collision mesh filename=package://spot_IL_environment/models/meshes/hl.hip.obj; visual mesh filename=package://spot_IL_environment/models/meshes/hl.hip.obj
- link hind_left.lowerleg: geometry collision mesh filename=package://spot_IL_environment/models/meshes/hl.lleg.obj; visual mesh filename=package://spot_IL_environment/models/meshes/hl.lleg.obj
- link hind_left.upperleg: geometry collision mesh filename=package://spot_IL_environment/models/meshes/hl.uleg.obj; visual mesh filename=package://spot_IL_environment/models/meshes/hl.uleg.obj
- link hind_right.hip: geometry collision mesh filename=package://spot_IL_environment/models/meshes/hr.hip.obj; visual mesh filename=package://spot_IL_environment/models/meshes/hr.hip.obj
- link hind_right.lowerleg: geometry collision mesh filename=package://spot_IL_environment/models/meshes/hr.lleg.obj; visual mesh filename=package://spot_IL_environment/models/meshes/hr.lleg.obj
- link hind_right.upperleg: geometry collision mesh filename=package://spot_IL_environment/models/meshes/hr.uleg.obj; visual mesh filename=package://spot_IL_environment/models/meshes/hr.uleg.obj

File: models/spot_box.urdf (robot description, URDF)
Before this commit: robot spot, 13 links, 12 joints
Links:
- link base_link: geometry collision mesh filename=package://spot_IL_environment/models/meshes/base.obj; visual mesh filename=package://spot_IL_environment/models/meshes/base.obj
- link front_left.hip: geometry collision mesh filename=package://spot_IL_environment/models/meshes/fl.hip.obj; visual mesh filename=package://spot_IL_environment/models/meshes/fl.hip.obj
- link front_left.lowerleg: geometry collision mesh filename=package://spot_IL_environment/models/meshes/fr.lleg.obj; visual mesh filename=package://spot_IL_environment/models/meshes/fr.lleg.obj
- link front_left.upperleg: geometry collision mesh filename=package://spot_IL_environment/models/meshes/fl.uleg.obj; visual mesh filename=package://spot_IL_environment/models/meshes/fl.uleg.obj
- link front_right.hip: geometry collision mesh filename=package://spot_IL_environment/models/meshes/fr.hip.obj; visual mesh filename=package://spot_IL_environment/models/meshes/fr.hip.obj
- link front_right.lowerleg: geometry collision mesh filename=package://spot_IL_environment/models/meshes/fr.lleg.obj; visual mesh filename=package://spot_IL_environment/models/meshes/fr.lleg.obj
- link front_right.upperleg: geometry collision mesh filename=package://spot_IL_environment/models/meshes/fr.uleg.obj; visual mesh filename=package://spot_IL_environment/models/meshes/fr.uleg.obj
- link hind_left.hip: geometry collision mesh filename=package://spot_IL_environment/models/meshes/hl.hip.obj; visual mesh filename=package://spot_IL_environment/models/meshes/hl.hip.obj
- link hind_left.lowerleg: geometry collision mesh filename=package://spot_IL_environment/models/meshes/hl.lleg.obj; visual mesh filename=package://spot_IL_environment/models/meshes/hl.lleg.obj
- link hind_left.upperleg: geometry collision mesh filename=package://spot_IL_environment/models/meshes/hl.uleg.obj; visual mesh filename=package://spot_IL_environment/models/meshes/hl.uleg.obj
- link hind_right.hip: geometry collision mesh filename=package://spot_IL_environment/models/meshes/hr.hip.obj; visual mesh filename=package://spot_IL_environment/models/meshes/hr.hip.obj
- link hind_right.lowerleg: geometry collision mesh filename=package://spot_IL_environment/models/meshes/hr.lleg.obj; visual mesh filename=package://spot_IL_environment/models/meshes/hr.lleg.obj
- link hind_right.upperleg: geometry collision mesh filename=package://spot_IL_environment/models/meshes/hr.uleg.obj; visual mesh filename=package://spot_IL_environment/models/meshes/hr.uleg.obj
