Commit message: Finalized the evaluation for rollout; Introduced the new format for defining worlds

File: models/spot/spot.urdf (robot description, URDF)
Before this commit: robot spot, 13 links, 12 joints
Links:
- link base_link: geometry collision mesh filename=package://spot_IL_environment/models/spot/meshes/base.obj; visual mesh filename=package://spot_IL_environment/models/spot/meshes/base.obj
- link front_left.hip: geometry collision mesh filename=package://spot_IL_environment/models/spot/meshes/fl.hip.obj; visual mesh filename=package://spot_IL_environment/models/spot/meshes/fl.hip.obj
- link front_left.lowerleg: geometry collision mesh filename=package://spot_IL_environment/models/spot/meshes/fr.lleg.obj; visual mesh filename=package://spot_IL_environment/models/spot/meshes/fr.lleg.obj
- link front_left.upperleg: geometry collision mesh filename=package://spot_IL_environment/models/spot/meshes/fl.uleg.obj; visual mesh filename=package://spot_IL_environment/models/spot/meshes/fl.uleg.obj
- link front_right.hip: geometry collision mesh filename=package://spot_IL_environment/models/spot/meshes/fr.hip.obj; visual mesh filename=package://spot_IL_environment/models/spot/meshes/fr.hip.obj
- link front_right.lowerleg: geometry collision mesh filename=package://spot_IL_environment/models/spot/meshes/fr.lleg.obj; visual mesh filename=package://spot_IL_environment/models/spot/meshes/fr.lleg.obj
- link front_right.upperleg: geometry collision mesh filename=package://spot_IL_environment/models/spot/meshes/fr.uleg.obj; visual mesh filename=package://spot_IL_environment/models/spot/meshes/fr.uleg.obj
- link hind_left.hip: geometry collision mesh filename=package://spot_IL_environment/models/spot/meshes/hl.hip.obj; visual mesh filename=package://spot_IL_environment/models/spot/meshes/hl.hip.obj
- link hind_left.lowerleg: geometry collision mesh filename=package://spot_IL_environment/models/spot/meshes/hl.lleg.obj; visual mesh filename=package://spot_IL_environment/models/spot/meshes/hl.lleg.obj
- link hind_left.upperleg: geometry collision mesh filename=package://spot_IL_environment/models/spot/meshes/hl.uleg.obj; visual mesh filename=package://spot_IL_environment/models/spot/meshes/hl.uleg.obj
- link hind_right.hip: geometry collision mesh filename=package://spot_IL_environment/models/spot/meshes/hr.hip.obj; visual mesh filename=package://spot_IL_environment/models/spot/meshes/hr.hip.obj
- link hind_right.lowerleg: geometry collision mesh filename=package://spot_IL_environment/models/spot/meshes/hr.lleg.obj; visual mesh filename=package://spot_IL_environment/models/spot/meshes/hr.lleg.obj
- link hind_right.upperleg: geometry collision mesh filename=package://spot_IL_environment/models/spot/meshes/hr.uleg.obj; visual mesh filename=package://spot_IL_environment/models/spot/meshes/hr.uleg.obj

File: models/spot/spot_box.urdf (robot description, URDF)
Before this commit: robot spot, 13 links, 12 joints
Links:
- link base_link: geometry collision mesh filename=package://spot_IL_environment/models/spot/meshes/base.obj; visual mesh filename=package://spot_IL_environment/models/spot/meshes/base.obj
- link front_left.hip: geometry collision mesh filename=package://spot_IL_environment/models/spot/meshes/fl.hip.obj; visual mesh filename=package://spot_IL_environment/models/spot/meshes/fl.hip.obj
- link front_left.lowerleg: geometry collision mesh filename=package://spot_IL_environment/models/spot/meshes/fr.lleg.obj; visual mesh filename=package://spot_IL_environment/models/spot/meshes/fr.lleg.obj
- link front_left.upperleg: geometry collision mesh filename=package://spot_IL_environment/models/spot/meshes/fl.uleg.obj; visual mesh filename=package://spot_IL_environment/models/spot/meshes/fl.uleg.obj
- link front_right.hip: geometry collision mesh filename=package://spot_IL_environment/models/spot/meshes/fr.hip.obj; visual mesh filename=package://spot_IL_environment/models/spot/meshes/fr.hip.obj
- link front_right.lowerleg: geometry collision mesh filename=package://spot_IL_environment/models/spot/meshes/fr.lleg.obj; visual mesh filename=package://spot_IL_environment/models/spot/meshes/fr.lleg.obj
- link front_right.upperleg: geometry collision mesh filename=package://spot_IL_environment/models/spot/meshes/fr.uleg.obj; visual mesh filename=package://spot_IL_environment/models/spot/meshes/fr.uleg.obj
- link hind_left.hip: geometry collision mesh filename=package://spot_IL_environment/models/spot/meshes/hl.hip.obj; visual mesh filename=package://spot_IL_environment/models/spot/meshes/hl.hip.obj
- link hind_left.lowerleg: geometry collision mesh filename=package://spot_IL_environment/models/spot/meshes/hl.lleg.obj; visual mesh filename=package://spot_IL_environment/models/spot/meshes/hl.lleg.obj
- link hind_left.upperleg: geometry collision mesh filename=package://spot_IL_environment/models/spot/meshes/hl.uleg.obj; visual mesh filename=package://spot_IL_environment/models/spot/meshes/hl.uleg.obj
- link hind_right.hip: geometry collision mesh filename=package://spot_IL_environment/models/spot/meshes/hr.hip.obj; visual mesh filename=package://spot_IL_environment/models/spot/meshes/hr.hip.obj
- link hind_right.lowerleg: geometry collision mesh filename=package://spot_IL_environment/models/spot/meshes/hr.lleg.obj; visual mesh filename=package://spot_IL_environment/models/spot/meshes/hr.lleg.obj
- link hind_right.upperleg: geometry collision mesh filename=package://spot_IL_environment/models/spot/meshes/hr.uleg.obj; visual mesh filename=package://spot_IL_environment/models/spot/meshes/hr.uleg.obj
